Commit message: Add files via upload

File: models/actuatorBot/actuatorFixedTop.urdf (robot description, URDF)
Before this commit: robot origins, 13 links, 12 joints
Links:
- link EE: geometry collision box size=0.001 0.001 0.001; visual box size=0.01 0.01 0.01
- link arml1: geometry collision box size=0.005 0.05 0.003; visual mesh filename=meshes/arm1.dae
- link arml2: geometry collision box size=0.005 0.05 0.003; visual mesh filename=meshes/arm1.dae
- link arml3: geometry collision box size=0.005 0.05 0.003; visual mesh filename=meshes/arm1.dae
- link arml4: geometry collision box size=0.005 0.05 0.003; visual mesh filename=meshes/arm1.dae
- link armr1: geometry collision box size=0.005 0.05 0.003; visual mesh filename=meshes/arm1.dae
- link armr2: geometry collision box size=0.005 0.05 0.003; visual mesh filename=meshes/arm1.dae
- link armr3: geometry collision box size=0.005 0.05 0.003; visual mesh filename=meshes/arm1.dae
- link armr4: geometry collision box size=0.005 0.05 0.003; visual mesh filename=meshes/arm1.dae
- link base_link: mass 10 -> 100; geometry collision mesh filename=meshes/baseALT.dae; visual mesh filename=meshes/baseALT.dae
- link carriage1: geometry collision box size=0.12 0.03 0.015; visual mesh filename=meshes/carriage.dae
- link carriage2: geometry collision box size=0.12 0.03 0.015; visual mesh filename=meshes/carriage.dae
- link middle: geometry collision box size=0.12 0.06 0.01; visual mesh filename=meshes/middle1.dae
Joints:
- joint arml1_to_middle: origin xyz=-0.0625 -0.045 0 rpy=0.3827 0 0 -> xyz=-0.0625 -0.045 0 rpy=0.7853981625 0 0
- joint base_to_carriage1: origin xyz=0 0.057 0.0075 -> xyz=0 0.045 0.0075
- joint base_to_carriage2: origin xyz=0 -0.057 0.0075 -> xyz=0 -0.045 0.0075
- joint carriage1_to_arml1: origin xyz=0.0625 0.008 0 rpy=-0.3827 0 0 -> xyz=0.0625 0.008 0 rpy=-0.7853981625 0 0
- joint carriage1_to_arml3: origin xyz=0.0625 -0.008 0 rpy=-0.3827 0 0 -> xyz=0.0625 -0.008 0 rpy=-0.7853981625 0 0
- joint carriage1_to_armr1: origin xyz=-0.0625 0.008 0 rpy=-0.3827 0 0 -> xyz=-0.0625 0.008 0 rpy=-0.7853981625 0 0
- joint carriage1_to_armr3: origin xyz=-0.0625 -0.008 0 rpy=-0.3827 0 0 -> xyz=-0.0625 -0.008 0 rpy=-0.7853981625 0 0
- joint carriage2_to_arml2: origin xyz=0.0625 0.008 0 rpy=0.3827 0 0 -> xyz=0.0625 0.008 0 rpy=0.7853981625 0 0
- joint carriage2_to_arml4: origin xyz=0.0625 -0.008 0 rpy=0.3827 0 0 -> xyz=0.0625 -0.008 0 rpy=0.7853981625 0 0
- joint carriage2_to_armr2: origin xyz=-0.0625 -0.008 0 rpy=0.3827 0 0 -> xyz=-0.0625 -0.008 0 rpy=0.7853981625 0 0
- joint carriage2_to_armr4: origin xyz=-0.0625 0.008 0 rpy=0.3827 0 0 -> xyz=-0.0625 0.008 0 rpy=0.7853981625 0 0

File: models/actuatorBot/actuatorFixedTop1.urdf (robot description, URDF)
Before this commit: robot origins, 13 links, 12 joints
Links:
- removed link EE
- removed link arml1
- removed link arml2
- removed link arml3
- removed link arml4
- removed link armr1
- removed link armr2
- removed link armr3
- removed link armr4
- removed link base_link
- removed link carriage1
- removed link carriage2
- removed link middle
- added link EE1; collision box size=0.001 0.001 0.001; visual box size=0.01 0.01 0.01
- added link arml11, mass 0.0159; collision box size=0.005 0.05 0.003; visual mesh filename=/meshes/arm1.dae
- added link arml21, mass 0.0159; collision box size=0.005 0.05 0.003; visual mesh filename=/meshes/arm1.dae
- added link arml31, mass 0.0159; collision box size=0.005 0.05 0.003; visual mesh filename=/meshes/arm1.dae
- added link arml41, mass 0.0159; collision box size=0.005 0.05 0.003; visual mesh filename=/meshes/arm1.dae
- added link armr11, mass 0.0159; collision box size=0.005 0.05 0.003; visual mesh filename=/meshes/arm1.dae
- added link armr21, mass 0.0159; collision box size=0.005 0.05 0.003; visual mesh filename=/meshes/arm1.dae
- added link armr31, mass 0.0159; collision box size=0.005 0.05 0.003; visual mesh filename=/meshes/arm1.dae
- added link armr41, mass 0.0159; collision box size=0.005 0.05 0.003; visual mesh filename=/meshes/arm1.dae
- added link base_link1, mass 100; collision mesh filename=/meshes/baseALT.dae; visual mesh filename=/meshes/baseALT.dae
- added link carriage11, mass 0.116; collision box size=0.12 0.03 0.015; visual mesh filename=/meshes/carriage.dae
- added link carriage21, mass 0.116; collision box size=0.12 0.03 0.015; visual mesh filename=/meshes/carriage.dae
- added link middle1, mass 0.07158; collision box size=0.12 0.06 0.01; visual mesh filename=/meshes/middle1.dae
Joints:
- removed joint arml1_to_middle
- removed joint base_to_carriage1
- removed joint base_to_carriage2
- removed joint carriage1_to_arml1
- removed joint carriage1_to_arml3
- removed joint carriage1_to_armr1
- removed joint carriage1_to_armr3
- removed joint carriage2_to_arml2
- removed joint carriage2_to_arml4
- removed joint carriage2_to_armr2
- removed joint carriage2_to_armr4
- removed joint middle_to_EE
- added joint arml1_to_middle1: type continuous, parent arml11, child middle1, origin xyz=-0.0625 -0.045 0 rpy=0.7853981625 0 0, axis 1 0 0
- added joint base_to_carriage11: type prismatic, parent base_link1, child carriage11, origin xyz=0 0.045 0.0075, axis 0 1 0, limit lower=-0.08 upper=.08 effort=1000.0 velocity=0.5
- added joint base_to_carriage21: type prismatic, parent base_link1, child carriage21, origin xyz=0 -0.045 0.0075, axis 0 1 0, limit lower=-0.08 upper=0.08 effort=1000.0 velocity=0.5
- added joint carriage1_to_arml11: type continuous, parent carriage11, child arml11, origin xyz=0.0625 0.008 0 rpy=-0.7853981625 0 0, axis 1 0 0
- added joint carriage1_to_arml31: type continuous, parent carriage11, child arml31, origin xyz=0.0625 -0.008 0 rpy=-0.7853981625 0 0, axis 1 0 0
- added joint carriage1_to_armr11: type continuous, parent carriage11, child armr11, origin xyz=-0.0625 0.008 0 rpy=-0.7853981625 0 0, axis 1 0 0
- added joint carriage1_to_armr31: type continuous, parent carriage11, child armr31, origin xyz=-0.0625 -0.008 0 rpy=-0.7853981625 0 0, axis 1 0 0
- added joint carriage2_to_arml21: type continuous, parent carriage21, child arml21, origin xyz=0.0625 0.008 0 rpy=0.7853981625 0 0, axis 1 0 0
- added joint carriage2_to_arml41: type continuous, parent carriage21, child arml41, origin xyz=0.0625 -0.008 0 rpy=0.7853981625 0 0, axis 1 0 0
- added joint carriage2_to_armr21: type continuous, parent carriage21, child armr21, origin xyz=-0.0625 -0.008 0 rpy=0.7853981625 0 0, axis 1 0 0
- added joint carriage2_to_armr41: type continuous, parent carriage21, child armr41, origin xyz=-0.0625 0.008 0 rpy=0.7853981625 0 0, axis 1 0 0
- added joint middle_to_EE1: type continuous, parent middle1, child EE1, origin xyz=0 -0.025 0.005 rpy=0 0 0, axis 0 0 1
